Commit message: 1.0.10

File: roch_description/urdf/roch.urdf.xacro (robot description, xacro)
@@ -105,16 +105,16 @@
 <!--        if not modify in gazebo will shack  -->
 <!--                                            -->
-<!--                                            -->
-<!--                                            -->
-<!--                                            -->
-<!--                                            -->
+<!--             Fixed this Bug                 -->
+<!--             Finally param                  -->
+<!--          L:0.13 0 -0.125                   -->
+<!--          R:-0.13 0 -0.0084                 -->
 <!--                                            -->
    <joint name="fornt_wheel_joint" type="fixed">
-      <origin xyz="0.13 0 -0.0084 " rpy="${-M_PI/2} 0 0" />
+      <origin xyz="0.13 0 -0.0125 " rpy="${-M_PI/2} 0 0" />
       <parent link="base_link" />
       <child link="front_wheel_link" />
    </joint>
    <joint name="rear_wheel_joint" type="fixed">
-      <origin xyz="-0.13 0 -0.008 " rpy="${-M_PI/2} 0 0" />
+      <origin xyz="-0.13 0 -0.0084 " rpy="${-M_PI/2} 0 0" />
       <parent link="base_link" />
       <child link="rear_wheel_link" />
@@ -133,33 +133,9 @@
     </link>
     <joint name="imu_joint" type="fixed">
-      <origin xyz="$(optenv HUSKY_IMU_XYZ 0.145 0 0.0095)" rpy="$(optenv HUSKY_IMU_RPY 0 -1.5708 3.1416)" />
+      <origin xyz=" 0.145 0 0.0095" rpy=" 0 -1.5708 3.1416" />
       <parent link="base_link" />
       <child link="imu_link" />
       <axis xyz="0 1 0"/>
     </joint>
-    <gazebo reference="imu_link">
-      <sensor type="imu" name="imu">
-      <always_on>true</always_on>
-      <update_rate>50</update_rate>
-      <visualize>false</visualize>
-        <imu>
-          <noise>
-            <type>gaussian</type>
-	          <rate>
-	            <mean>0.0</mean>
-	            <stddev>${0.0014*0.0014}</stddev> <!-- 0.25 x 0.25 (deg/s) -->
-	            <bias_mean>0.0</bias_mean>
-	            <bias_stddev>0.0</bias_stddev>
-	          </rate>
-		        <accel> <!-- not used in the plugin and real robot, hence using tutorial values -->
-			        <mean>0.0</mean>
-			        <stddev>1.7e-2</stddev>
-			        <bias_mean>0.1</bias_mean>
-			        <bias_stddev>0.001</bias_stddev>
-		        </accel>
-          </noise>
-	      </imu>
-      </sensor>
-    </gazebo>
     <xacro:roch_ultrasonic ultrasonic_prefix="front_left" parent="base_link">
       <origin xyz="0.1631 0.06756 0.123" rpy="0 ${-M_PI/2} 0" />
@@ -188,27 +164,4 @@
  <!-- roch Gazebo simulation details -->
   <roch_robot_gazebo/>
- <!-- laser model
-  <xacro:if value="$(arg laser_enabled)">
-      <joint name="base_laser_mount" type="fixed">
-        <origin xyz="0.001 0 0.1" rpy="0 0 0" />
-        <parent link="base_link" />
-        <child link="base_laser" />
-      </joint>
-      <xacro:sick_lms100 prefix="base" />
-  </xacro:if>  -->
-  <!-- Husky kinect macros
-   <xacro:if value="$(arg kinect_enabled)">
-      <joint name="kinect_frame_joint" type="fixed">
-        <origin xyz="$(optenv HUSKY_KINECT_XYZ 0.09 0 0.072)" rpy="$(optenv HUSKY_KINECT_RPY 0 0 0)" />
-        <parent link="base_link"/>
-        <child link="camera_link"/>
-      </joint>
-      <xacro:kinect_camera prefix="camera"/>
-   </xacro:if> -->
-  <!-- asus xtion model
-  <xacro:if value="$(arg asus_xtion_enabled)">
-     <sensor_asus_xtion_pro parent="base_link"/>
-  </xacro:if>   -->
-<!-- -->
 </xacro:macro>
 </robot>

File: roch_description/urdf/roch_gazebo.urdf.xacro (robot description, xacro)
@@ -40,4 +40,38 @@
     </gazebo>
   </xacro:macro>
+  <xacro:macro name="roch_sim_2dlaser">
+    <gazebo reference="base_laser">
+      <turnGravityOff>true</turnGravityOff>
+      <sensor type="ray" name="laser">
+        <pose>0 0 0 0 0 0</pose>
+        <visualize>false</visualize>
+        <update_rate>50</update_rate>
+        <ray>
+          <scan>
+            <horizontal>
+              <samples>720</samples>
+              <resolution>1</resolution>
+              <min_angle>-2.35619</min_angle>
+              <max_angle>2.35619</max_angle>
+            </horizontal>
+          </scan>
+          <range>
+            <min>0.10</min>
+            <max>30.0</max>
+            <resolution>0.01</resolution>
+          </range>
+          <noise>
+            <type>gaussian</type>
+            <mean>0.0</mean>
+            <stddev>0.001</stddev>
+          </noise>
+        </ray>
+        <plugin name="gazebo_ros_laser" filename="libgazebo_ros_laser.so">
+          <topicName>scan</topicName>
+          <frameName>base_laser</frameName>
+        </plugin>
+      </sensor>
+    </gazebo>
+  </xacro:macro>
  <!-- roch imu/gps controller for simulation -->
   <xacro:macro name="roch_robot_gazebo">
@@ -74,4 +108,34 @@
       </plugin>
     </gazebo>
+    <gazebo reference="imu_link">
+      <sensor type="imu" name="imu">
+      <always_on>true</always_on>
+      <update_rate>50</update_rate>
+      <visualize>false</visualize>
+        <imu>
+          <noise>
+            <type>gaussian</type>
+	          <rate>
+	            <mean>0.0</mean>
+	            <stddev>${0.0014*0.0014}</stddev> <!-- 0.25 x 0.25 (deg/s) -->
+	            <bias_mean>0.0</bias_mean>
+	            <bias_stddev>0.0</bias_stddev>
+	          </rate>
+		        <accel> <!-- not used in the plugin and real robot, hence using tutorial values -->
+			        <mean>0.0</mean>
+			        <stddev>1.7e-2</stddev>
+			        <bias_mean>0.1</bias_mean>
+			        <bias_stddev>0.001</bias_stddev>
+		        </accel>
+          </noise>
+	      </imu>
+      </sensor>
+    </gazebo>
+    <!-- Gazebo plugin for ROS Control -->
+    <gazebo>
+      <plugin name="gazebo_ros_control" filename="libgazebo_ros_control.so">
+        <robotNamespace>/</robotNamespace>
+      </plugin>
+    </gazebo>
 <!--
     <gazebo>

File: roch_description/urdf/sensors/ls_ls01c.urdf.xacro (robot description, xacro)
@@ -26,4 +26,6 @@
 -->
 <robot xmlns:xacro="http://ros.org/wiki/xacro" name="ls_ls01c">
+  <xacro:include filename="$(find roch_description)/urdf/roch_gazebo.urdf.xacro"/>
+  <xacro:include filename="$(find roch_description)/urdf/roch_properties.urdf.xacro"/>
   <xacro:property name="laser_x" value="0.08" />
   <xacro:property name="laser_y" value="0.08" />
@@ -64,36 +66,6 @@
       <child link="base_laser" />
     </joint>
-    <gazebo reference="base_laser">
-      <turnGravityOff>true</turnGravityOff>
-      <sensor type="ray" name="laser">
-        <pose>0 0 0 0 0 0</pose>
-        <visualize>false</visualize>
-        <update_rate>50</update_rate>
-        <ray>
-          <scan>
-            <horizontal>
-              <samples>720</samples>
-              <resolution>1</resolution>
-              <min_angle>-2.35619</min_angle>
-              <max_angle>2.35619</max_angle>
-            </horizontal>
-          </scan>
-          <range>
-            <min>0.10</min>
-            <max>30.0</max>
-            <resolution>0.01</resolution>
-          </range>
-          <noise>
-            <type>gaussian</type>
-            <mean>0.0</mean>
-            <stddev>0.001</stddev>
-          </noise>
-        </ray>
-        <plugin name="gazebo_ros_laser" filename="libgazebo_ros_laser.so">
-          <topicName>scan</topicName>
-          <frameName>base_laser</frameName>
-        </plugin>
-      </sensor>
-    </gazebo>
+    <!-- 2d laser for simulation, same as rplidar -->
+    <roch_sim_2dlaser/>
   </xacro:macro>
 </robot>

File: roch_description/urdf/sensors/rplidar.urdf.xacro (robot description, xacro)
@@ -26,4 +26,6 @@
 -->
 <robot xmlns:xacro="http://ros.org/wiki/xacro" name="rplidar">
+  <xacro:include filename="$(find roch_description)/urdf/roch_gazebo.urdf.xacro"/>
+  <xacro:include filename="$(find roch_description)/urdf/roch_properties.urdf.xacro"/>
   <xacro:property name="laser_x" value="0.08" />
   <xacro:property name="laser_y" value="0.08" />
@@ -64,36 +66,6 @@
       <child link="base_laser" />
     </joint>
-    <gazebo reference="base_laser">
-      <turnGravityOff>true</turnGravityOff>
-      <sensor type="ray" name="laser">
-        <pose>0 0 0 0 0 0</pose>
-        <visualize>false</visualize>
-        <update_rate>50</update_rate>
-        <ray>
-          <scan>
-            <horizontal>
-              <samples>720</samples>
-              <resolution>1</resolution>
-              <min_angle>-2.35619</min_angle>
-              <max_angle>2.35619</max_angle>
-            </horizontal>
-          </scan>
-          <range>
-            <min>0.10</min>
-            <max>30.0</max>
-            <resolution>0.01</resolution>
-          </range>
-          <noise>
-            <type>gaussian</type>
-            <mean>0.0</mean>
-            <stddev>0.001</stddev>
-          </noise>
-        </ray>
-        <plugin name="gazebo_ros_laser" filename="libgazebo_ros_laser.so">
-          <topicName>scan</topicName>
-          <frameName>base_laser</frameName>
-        </plugin>
-      </sensor>
-    </gazebo>
+    <!-- 2d laser for simulation, same as rplidar -->
+    <roch_sim_2dlaser/>
   </xacro:macro>
 </robot>

Commit message: Update roch.urdf.xacro

File: roch_description/urdf/roch.urdf.xacro (robot description, xacro)
@@ -136,5 +136,4 @@
       <parent link="base_link" />
       <child link="imu_link" />
-      <axis xyz="0 1 0"/>
     </joint>
     <xacro:roch_ultrasonic ultrasonic_prefix="front_left" parent="base_link">

Commit message: Update rplidar position and imu in Roch.

File: roch_description/urdf/roch.urdf.xacro (robot description, xacro)
@@ -133,7 +133,8 @@
     </link>
     <joint name="imu_joint" type="fixed">
-      <origin xyz=" 0.145 0 0.0095" rpy=" 0 -1.5708 3.1416" />
+      <origin xyz=" 0.145 0 0.0095" rpy=" 0 0 3.1415926" />
       <parent link="base_link" />
       <child link="imu_link" />
+      <axis xyz="0 1 0"/>
     </joint>
     <xacro:roch_ultrasonic ultrasonic_prefix="front_left" parent="base_link">
