Commit message: Support sick lms100.

File: roch_description/urdf/roch_gazebo.urdf.xacro (robot description, xacro)
@@ -70,4 +70,40 @@
           <topicName>scan</topicName>
           <frameName>base_laser</frameName>
+        </plugin>
+      </sensor>
+    </gazebo>
+  </xacro:macro>
+  <xacro:macro name="roch_sim_2dlaser_custom"  params="frame:=laser topic:=scan sample_size:=720 update_rate:=50
+               min_angle:=-2.35619 max_angle:=2.35619 min_range:=0.1 max_range:=30.0 robot_namespace:=/">
+    <gazebo reference="${frame}">
+      <turnGravityOff>true</turnGravityOff>
+      <sensor type="ray" name="${frame}">
+        <pose>0 0 0 0 0 0</pose>
+        <visualize>false</visualize>
+        <update_rate>${update_rate}</update_rate>
+        <ray>
+          <scan>
+            <horizontal>
+              <samples>${sample_size}</samples>
+              <resolution>1</resolution>
+              <min_angle>${min_angle}</min_angle>
+              <max_angle>${max_angle}</max_angle>
+            </horizontal>
+          </scan>
+          <range>
+            <min>${min_range}</min>
+            <max>${max_range}</max>
+            <resolution>0.01</resolution>
+          </range>
+          <noise>
+            <type>gaussian</type>
+            <mean>0.0</mean>
+            <stddev>0.001</stddev>
+          </noise>
+        </ray>
+        <plugin name="gazebo_ros_laser" filename="libgazebo_ros_laser.so">
+          <topicName>${topic}</topicName>
+          <frameName>${frame}</frameName>
+          <robotNamespace>${robot_namespace}</robotNamespace>
         </plugin>
       </sensor>

File: roch_description/urdf/roch_library.urdf.xacro (robot description, xacro)
@@ -21,3 +21,4 @@
   <xacro:include filename="$(find roch_description)/urdf/sensors/ls_ls01c.urdf.xacro"/>
   <xacro:include filename="$(find roch_description)/urdf/sensors/rplidar.urdf.xacro"/>
+  <xacro:include filename="$(find roch_description)/urdf/sensors/sick_lmsxx.urdf.xacro"/>
 </robot>

Commit message: update

File: roch_description/urdf/roch_gazebo.urdf.xacro (robot description, xacro)
@@ -70,40 +70,4 @@
           <topicName>scan</topicName>
           <frameName>base_laser</frameName>
-        </plugin>
-      </sensor>
-    </gazebo>
-  </xacro:macro>
-  <xacro:macro name="roch_sim_2dlaser_custom"  params="frame:=laser topic:=scan sample_size:=720 update_rate:=50
-               min_angle:=-2.35619 max_angle:=2.35619 min_range:=0.1 max_range:=30.0 robot_namespace:=/">
-    <gazebo reference="${frame}">
-      <turnGravityOff>true</turnGravityOff>
-      <sensor type="ray" name="${frame}">
-        <pose>0 0 0 0 0 0</pose>
-        <visualize>false</visualize>
-        <update_rate>${update_rate}</update_rate>
-        <ray>
-          <scan>
-            <horizontal>
-              <samples>${sample_size}</samples>
-              <resolution>1</resolution>
-              <min_angle>${min_angle}</min_angle>
-              <max_angle>${max_angle}</max_angle>
-            </horizontal>
-          </scan>
-          <range>
-            <min>${min_range}</min>
-            <max>${max_range}</max>
-            <resolution>0.01</resolution>
-          </range>
-          <noise>
-            <type>gaussian</type>
-            <mean>0.0</mean>
-            <stddev>0.001</stddev>
-          </noise>
-        </ray>
-        <plugin name="gazebo_ros_laser" filename="libgazebo_ros_laser.so">
-          <topicName>${topic}</topicName>
-          <frameName>${frame}</frameName>
-          <robotNamespace>${robot_namespace}</robotNamespace>
         </plugin>
       </sensor>

File: roch_description/urdf/roch_library.urdf.xacro (robot description, xacro)
@@ -21,4 +21,3 @@
   <xacro:include filename="$(find roch_description)/urdf/sensors/ls_ls01c.urdf.xacro"/>
   <xacro:include filename="$(find roch_description)/urdf/sensors/rplidar.urdf.xacro"/>
-  <xacro:include filename="$(find roch_description)/urdf/sensors/sick_lmsxx.urdf.xacro"/>
 </robot>

File: roch_description/urdf/sensors/rplidar.urdf.xacro (robot description, xacro)
@@ -3,5 +3,5 @@
 Copyright (c) 2013, Goncalo Cabrita, ISR University of Coimbra
 Copyright (c) 2014, Clearpath Robotics
-Copyright (c) 2016, Soy Robotics
+Copyright (c) 2016, SawYer Robotics
 All rights reserved.
 Redistribution and use in source and binary forms, with or without
